Commit message: Modif - Xacros - ArUco Markers 6x6 OpenCV

File: xacro/iris2.xacro (robot description, xacro)
@@ -5,5 +5,5 @@
   <xacro:property name="rotor_velocity_slowdown_sim" value="10" />
   <xacro:property name="use_mesh_file" value="true" />
-  <xacro:property name="mesh_file" value="package://rotors_description/meshes/iris.dae" />
+  <xacro:property name="mesh_file" value="package://vc_new_controller/meshes/iris2.dae" />
   <xacro:property name="mass" value="1.5" /> <!-- [kg] -->
   <xacro:property name="body_width" value="0.47" /> <!-- [m] -->

File: xacro/iris3.xacro (robot description, xacro)
@@ -5,5 +5,5 @@
   <xacro:property name="rotor_velocity_slowdown_sim" value="10" />
   <xacro:property name="use_mesh_file" value="true" />
-  <xacro:property name="mesh_file" value="package://rotors_description/meshes/iris.dae" />
+  <xacro:property name="mesh_file" value="package://vc_new_controller/meshes/iris3.dae" />
   <xacro:property name="mass" value="1.5" /> <!-- [kg] -->
   <xacro:property name="body_width" value="0.47" /> <!-- [m] -->
@@ -28,9 +28,11 @@
   <!-- Property Blocks -->
   <xacro:property name="body_inertia">
-    <inertia ixx="0.0347563" ixy="0.0" ixz="0.0" iyy="0.0458929" iyz="0.0" izz="0.0977" /> <!-- [kg.m^2] [kg.m^2] [kg.m^2] [kg.m^2] [kg.m^2] [kg.m^2] -->
+    <inertia ixx="0.0347563" ixy="0.0" ixz="0.0" iyy="0.0458929" iyz="0.0" izz="0.0977" /> <!--
+    [kg.m^2] [kg.m^2] [kg.m^2] [kg.m^2] [kg.m^2] [kg.m^2] -->
   </xacro:property>
   <!-- inertia of a single rotor, assuming it is a cuboid. Height=3mm, width=15mm -->
   <xacro:property name="rotor_inertia">
-    <xacro:box_inertia x="${radius_rotor}" y="0.015" z="0.003" mass="${mass_rotor*rotor_velocity_slowdown_sim}" />
+    <xacro:box_inertia x="${radius_rotor}" y="0.015" z="0.003"
+      mass="${mass_rotor*rotor_velocity_slowdown_sim}" />
   </xacro:property>
   <!-- Included URDF Files -->
@@ -44,5 +46,5 @@
     use_mesh_file="${use_mesh_file}"
     mesh_file="${mesh_file}"
-    >
+  >
     <xacro:insert_block name="body_inertia" />
   </xacro:multirotor_base_macro>
@@ -130,4 +132,5 @@
     <xacro:insert_block name="rotor_inertia" />
   </xacro:vertical_rotor>
+  <!-- Initialized cameras in front and bottom -->
   <xacro:camera_macro
     namespace="${namespace}"
@@ -144,8 +147,8 @@
     noise_stddev="0.007"
     enable_visual="true">
-      <box size="0.05 0.05 0.02" />
-      <origin xyz="0 0 -0.03" rpy="0 1.570796 0" />
+    <box size="0.05 0.05 0.02" />
+    <origin xyz="0 0 -0.03" rpy="0 1.570796 0" />
   </xacro:camera_macro>
-  <!--<xacro:camera_macro
+  <xacro:camera_macro
     namespace="${namespace}"
     parent_link="${namespace}/base_link"
@@ -161,6 +164,6 @@
     noise_stddev="0.007"
     enable_visual="true">
-      <box size="0.05 0.05 0.02" />
-      <origin xyz="0.09 0 0" rpy="0 0 0" />
-  </xacro:camera_macro>-->
+    <box size="0.05 0.05 0.02" />
+    <origin xyz="0.09 0 0" rpy="0 0 0" />
+  </xacro:camera_macro>
 </robot>
